File: redox/pcb/rev1.0/kicad_files/redox_rev1.kicad_pcb (KiCad board)
At the start: 2 copper layers, 162.2 x 126.5 mm, 86 parts, among them K0 KEYSW, K1 KEYSW, K10 KEYSW, K11 KEYSW, K12 KEYSW, K13 KEYSW, K14 KEYSW, K15 KEYSW, K16 KEYSW, K2 KEYSW, K20 KEYSW, K21 KEYSW, K22 KEYSW, K23 KEYSW, K24 KEYSW, K25 KEYSW, K26 KEYSW, K3 KEYSW, K30 KEYSW, K31 KEYSW, K32 KEYSW, K33 KEYSW, K34 KEYSW, K35 KEYSW, K36 KEYSW, K4 KEYSW, K40 KEYSW, K41 KEYSW, K42 KEYSW, K43 KEYSW, K44 KEYSW, K45 KEYSW, K46 KEYSW, K5 KEYSW, K6 KEYSW, U1 ProMicro

Commit message: design updates
Parts:
- removed the G*** at (102.2, 102.9)
- removed the G*** at (102.2, 102.2)
- K0, K10, K20, K30: footprint myparts:Mx_Alps_125-dualside -> Keebio-Parts:Mx_Alps_100-dualside
- K16: footprint canadian_footprints:Mx_Alps_150-dualsided -> Keebio-Parts:Mx_Alps_100-dualside
- moved K16 19.9 mm to (208.3, 77.9), turned to 0 degrees
- moved D0 15.0 mm to (94.0, 60.1)
- moved D10 15.0 mm to (94.0, 79.2)
- moved D30 15.0 mm to (94.0, 117.3)
- moved K20 15.0 mm to (94.0, 90.0)
- moved K30 15.0 mm to (94.0, 109.0)
- moved D20 15.0 mm to (94.0, 98.2)
- moved K0 15.0 mm to (94.0, 51.9)
- moved K10 15.0 mm to (94.0, 70.9)
- moved D1 14.8 mm to (113.0, 60.1)
- moved D11 14.8 mm to (113.0, 79.2)
- moved D13 14.8 mm to (151.1, 72.2)
- moved D16 14.8 mm to (208.3, 91.9)
- moved D26 14.8 mm to (207.6, 119.8)
- moved D31 14.8 mm to (113.0, 117.3)
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Routing:
- net col6: track 184.3 -> 161.1 mm
- net Net-(D16-Pad2): track 5.88 -> 18.5 mm
- net col0: track 167.6 -> 172.4 mm
- net row2: track 188.9 -> 186.3 mm
- net row3: track 207.9 -> 205.2 mm
- net row1: track 169.3 -> 166.6 mm
- net row0: track 135.3 -> 132.8 mm
Other:
- board size 162.2 x 126.5 mm -> 161.8 x 126.2 mm
- net class Default removed
- board text added: "Redesigned by 3DG-Tech"
- board text removed: "designed by Mattia Dal Ben (https://github.com/mattdibi)"
